File: RAM.sch (KiCad schematic (older format))
At the start: 27 parts, among them IC1 EP4CE10F17, U22 W9751G6KB

Commit message: More bottom length matching
Parts:
- gave numbers to parts that had none: 4
Changed lines of the file:
@@
 BA1
 $Comp
-L GND #PWR131
+L GND #PWR0131
 U 1 1 5882F59D
 P 6275 7300
-F 0 "#PWR131" H 6275 7050 50  0001 C CNN
+F 0 "#PWR0131" H 6275 7050 50  0001 C CNN
 F 1 "GND" H 6275 7150 50  0001 C CNN
 F 2 "" H 6275 7300 50  0000 C CNN
@@
 Text Label 5250 2350 2    50   ~ 0
 A9
-Text Label 7950 3325 2    50   ~ 0
+Text Label 7950 1825 2    50   ~ 0
 CLK_N
-Text Label 7950 3400 2    50   ~ 0
+Text Label 7950 1900 2    50   ~ 0
 CLK_P
 Text Label 7950 1975 2    50   ~ 0
@@
 Text Label 7950 2050 2    50   ~ 0
 A0
-Text Label 7950 1825 2    50   ~ 0
+Text Label 7950 3400 2    50   ~ 0
 CS#
 Text Label 5250 2125 2    50   ~ 0
@@
 +1V8
 $Comp
-L GND #PWR132
+L GND #PWR0132
 U 1 1 5883C563
 P 6950 5300
-F 0 "#PWR132" H 6950 5050 50  0001 C CNN
+F 0 "#PWR0132" H 6950 5050 50  0001 C CNN
 F 1 "GND" H 6950 5150 50  0001 C CNN
 F 2 "" H 6950 5300 50  0000 C CNN
@@
 $EndComp
 $Comp
-L GND #PWR133
+L GND #PWR0133
 U 1 1 5883EF35
 P 6950 5925
-F 0 "#PWR133" H 6950 5675 50  0001 C CNN
+F 0 "#PWR0133" H 6950 5675 50  0001 C CNN
 F 1 "GND" H 6950 5775 50  0001 C CNN
 F 2 "" H 6950 5925 50  0000 C CNN
@@
 	8350 5925 8350 5875
 $Comp
-L C_Small C?
+L C_Small C94
 U 1 1 5884E5C8
 P 8550 5775
-F 0 "C?" H 8560 5845 50  0000 L CNN
+F 0 "C94" H 8560 5845 50  0000 L CNN
 F 1 "0,1" H 8560 5695 50  0000 L CNN
 F 2 "Capacitors_SMD:C_0402" H 8550 5775 25  0000 C CNN
@@
 $EndComp
 $Comp
-L C_Small C?
+L C_Small C95
 U 1 1 5884E5CE
 P 8750 5775
-F 0 "C?" H 8760 5845 50  0000 L CNN
+F 0 "C95" H 8760 5845 50  0000 L CNN
 F 1 "0,1" H 8760 5695 50  0000 L CNN
 F 2 "Capacitors_SMD:C_0402" H 8750 5775 25  0000 C CNN
@@
 $EndComp
 $Comp
-L C_Small C?
+L C_Small C96
 U 1 1 5884E5D4
 P 8950 5775
-F 0 "C?" H 8960 5845 50  0000 L CNN
+F 0 "C96" H 8960 5845 50  0000 L CNN
 F 1 "0,1" H 8960 5695 50  0000 L CNN
 F 2 "Capacitors_SMD:C_0402" H 8950 5775 25  0000 C CNN
@@
 $EndComp
 $Comp
-L C_Small C?
+L C_Small C97
 U 1 1 5884E5DA
 P 9150 5775
-F 0 "C?" H 9160 5845 50  0000 L CNN
+F 0 "C97" H 9160 5845 50  0000 L CNN
 F 1 "0,1" H 9160 5695 50  0000 L CNN
 F 2 "Capacitors_SMD:C_0402" H 9150 5775 25  0000 C CNN

Commit message: Cleanups
Connections:
- wire segments 132 -> 157
Other:
- moved on the sheet: C73, C74, C75, C76, C77, C78, C79, C80, C81, C82, C83, C84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

Commit message: More tuning
Changed lines of the file:
@@
 Text Label 6625 1175 2    50   ~ 0
 DQ10
-Text Label 6625 1700 2    50   ~ 0
+Text Label 6625 2225 2    50   ~ 0
 A8
-Text Label 6625 2225 2    50   ~ 0
-A11
 Text Label 3950 1275 2    50   ~ 0
 A9
@@
 Wire Wire Line
 	9350 5000 9350 5050
+Text Label 6625 1700 2    50   ~ 0
+A11
 $EndSCHEMATC
